File: keyboards/eyeohdesigns/theboulevard/PCBFiles/mainpcb/theboulevard.kicad_pcb (KiCad board)
At the start: 2 copper layers, 257.2 x 85.7 mm, 157 parts, among them J1 Conn_01x04_Female, J2 Conn_01x12_Male, K1 KEYSW, K10 KEYSW, K11 KEYSW, K12 KEYSW, K13 KEYSW, K14 KEYSW, K151 KEYSW, K152 KEYSW, K161 KEYSW, K162 KEYSW, K171 KEYSW, K172 KEYSW, K181 KEYSW, K182 KEYSW, K191 KEYSW, K192 KEYSW, K2 KEYSW, K201 KEYSW, K202 KEYSW, K211 KEYSW, K212 KEYSW, K221 KEYSW, K222 KEYSW, K231 KEYSW, K232 KEYSW, K241 KEYSW, K242 KEYSW, K25 KEYSW, K261 KEYSW, K262 KEYSW, K27 KEYSW, K281 KEYSW, K282 KEYSW, K291 KEYSW, K3 KEYSW, K301 KEYSW, K302 KEYSW, K311 KEYSW, K312 KEYSW, K321 KEYSW, K322 KEYSW, K331 KEYSW, K332 KEYSW, K341 KEYSW, K342 KEYSW, K351 KEYSW, K352 KEYSW, K361 KEYSW, K362 KEYSW, K371 KEYSW, K372 KEYSW, K381 KEYSW, K382 KEYSW, K391 KEYSW, K392 KEYSW, K4 KEYSW, K40 KEYSW, K411 KEYSW, K412 KEYSW, K421 KEYSW, K422 KEYSW, K431 KEYSW, K432 KEYSW, K44 KEYSW, K451 KEYSW, K452 KEYSW, K453 KEYSW, K461 KEYSW, K462 KEYSW, K471 KEYSW, K472 KEYSW, K473 KEYSW, K481 KEYSW, K482 KEYSW, K483 KEYSW, K49 KEYSW, K5 KEYSW, K501 KEYSW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

Commit message: Fixes a reversed connector on the main PCB
Parts:
- removed the REF** at (36.8, 83.2) (x2)
- moved C5 41.7 mm to (39.2, 24.8), turned to 0 degrees
Connections:
- J1 pad 1: GND -> VCC
- J1 pad 4: VCC -> GND
- R1 pad 2: Net-(J1-Pad3) -> Net-(J1-Pad2)
- R2 pad 2: Net-(J1-Pad2) -> Net-(J1-Pad3)
Routing:
- net VCC: track 242.1 -> 262.0 mm
- net Net-(J1-Pad3): track 39.8 -> 32.6 mm
- net /Col11: track 344.3 -> 341.5 mm
- net /Col10: track 311.9 -> 310.2 mm
- net /Col12: track 389.2 -> 388.1 mm
- net GND: track 39.1 -> 39.9 mm, vias 10 -> 13
