File: keyboards/eyeohdesigns/theboulevard/PCBFiles/mainpcb/theboulevard.sch (KiCad schematic (older format))
At the start: 154 parts, among them J1 Conn_01x04_Female, J2 Conn_01x12_Male, K1 KEYSW, K10 KEYSW, K11 KEYSW, K12 KEYSW, K13 KEYSW, K14 KEYSW, K151 KEYSW, K152 KEYSW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

Commit message: Fixes a reversed connector on the main PCB
Connections:
- wire segments 266 -> 255
- no-connect marks 1 -> 0
Other:
- moved on the sheet: R1, R2
